Commit message: Fixed bug where the base_link x-axis was to the left of the robot

File: urdf/my_robot.urdf.xacro (robot description, xacro)
@@ -2,9 +2,4 @@
 <robot name="jo_bot" xmlns:xacro="http://ros.org/wiki/xacro">
   <xacro:include filename="$(find my_robot_description)/urdf/my_robot.gazebo" />
-  <link name="base_footprint" />
-  <joint name="base_footprint_joint" type="fixed">
-    <parent link="base_footprint" />
-    <child link="base_link" />
-  </joint>
   <xacro:property name="pi" value="3.1415926535897931" />
   <xacro:property name="base_width" value="0.1" />
@@ -62,4 +57,10 @@
     </inertial>
   </xacro:macro>
+  <link name="base_footprint" />
+  <joint name="base_footprint_joint" type="fixed">
+    <parent link="base_footprint" />
+    <child link="base_link" />
+    <origin xyz="0 0 0" rpy="0 0 ${-pi / 2}" />
+  </joint>
   <link name="base_link">
     <visual>
